Commit message: moveit whole body planning for raw31

File: cob_hardware_config/cob4-2/urdf/cob4-2.urdf.xacro (robot description, xacro)
@@ -18,6 +18,6 @@
   <!-- head -->
   <xacro:include filename="$(find cob_description)/urdf/cob4_head/head.urdf.xacro" />
-  <!-- sensorring -->
-  <xacro:include filename="$(find cob_description)/urdf/cob4_sensorring/sensorring_asus.urdf.xacro" />
+  <!-- sensorring
+  <xacro:include filename="$(find cob_description)/urdf/cob4_sensorring/sensorring_asus.urdf.xacro" /> -->
   <!-- composition of the robot -->
   <xacro:base name="base" use_old_joint_names="false"/>
@@ -46,4 +46,5 @@
     </plugin>
   </gazebo>
+<!--
   <xacro:sensorring name="sensorring" parent="head_3_link">
     <origin xyz="${sensorring_x} ${sensorring_y} ${sensorring_z}" rpy="${sensorring_roll} ${sensorring_pitch} ${sensorring_yaw}" />
@@ -55,4 +56,5 @@
     </plugin>
   </gazebo>
+-->
   <xacro:schunk_lwa4p_extended name="arm_right" parent="torso_3_link" has_podest="false">
     <origin xyz="${arm_right_x} ${arm_right_y} ${arm_right_z}" rpy="${arm_right_roll} ${arm_right_pitch} ${arm_right_yaw}" />

File: cob_hardware_config/raw3-1/urdf/raw3-1.urdf.xacro (robot description, xacro)
@@ -22,4 +22,10 @@
   <xacro:include filename="$(find raw_description)/urdf/vacuum_gripper/gripper.urdf.xacro"/>
   <xacro:property name="arm_prefix" value="arm_"/>
+  <link name="odom_combined"/>
+  <joint name="world_to_stand" type="planar">
+    <parent link="odom_combined"/>
+	<child link="base_footprint"/>
+	<origin xyz="-0.238 0 0"/>
+  </joint>
   <!-- composition of the robot -->
   <xacro:raw_base name="base"/>
@@ -69,5 +75,5 @@
     <origin xyz="${gripper_x} ${gripper_y} ${gripper_z}" rpy="0 0 0" />
   </xacro:vacuum_gripper_definition>
-  <!-- IMU brick mount on raw3-1 -->
+  <!-- IMU brick mount on raw3-1
   <joint name="imu_brick_joint" type="fixed" >
     <origin xyz="0.402 -0.0811 0.335" rpy="0 0 0" />
@@ -84,5 +90,5 @@
       <material name="IPA/LightGrey" />
     </visual>
-  </link>
+  </link>-->
   <!-- END: IMU brick  mount -->
   <!-- rfid_front mount on raw3-1 -->
