Commit message: whole body moveit configuration with virtual joint working

File: cob_hardware_config/raw3-1-2/urdf/raw3-1-2.urdf.xacro (robot description, xacro)
@@ -1,6 +1,6 @@
 <?xml version="1.0" ?>
 <robot name="raw3-1-2" xmlns:xacro="http://ros.org/wiki/xacro">
-  <xacro:include filename="$(find ipa_order_picking_arm_planning)/robot_conf/urdf/raw3-1.urdf.xacro" />
-  <!--virtual_joint name="world_joint" type="planar" parent_frame="odom_combined" child_link="base_footprint"/ -->
+  <!--xacro:include filename="$(find ipa_order_picking_arm_planning)/robot_conf/urdf/raw3-1.urdf.xacro" /> -->
+  <xacro:include filename="$(find cob_hardware_config)/raw3-1/urdf/raw3-1.urdf.xacro" />
   <xacro:macro name="raw3-1"/>
 </robot>

File: cob_hardware_config/raw3-1/urdf/model.urdf (robot description, URDF)
Before this commit: robot raw3-1, 40 links, 39 joints
Links:
- removed link odom_combined
Joints:
- removed joint world_to_stand

File: cob_hardware_config/raw3-1/urdf/raw3-1.urdf.xacro (robot description, xacro)
@@ -22,10 +22,4 @@
   <xacro:include filename="$(find raw_description)/urdf/vacuum_gripper/gripper.urdf.xacro"/>
   <xacro:property name="arm_prefix" value="arm_"/>
-  <link name="odom_combined"/>
-  <joint name="world_to_stand" type="planar">
-    <parent link="odom_combined"/>
-	<child link="base_footprint"/>
-	<origin xyz="-0.238 0 0"/>
-  </joint>
   <!-- composition of the robot -->
   <xacro:raw_base name="base"/>
