Commit message: new gripper position

File: cob_hardware_config/robots/raw3-1/urdf/calibration_default.urdf.xacro (robot description, xacro)
@@ -53,5 +53,5 @@
 	<xacro:property name="def_gripper_y" value="0.0"/>
 	<xacro:property name="def_gripper_z" value="0.0"/>
-	<xacro:property name="def_gripper_roll" value="0.0"/>
+	<xacro:property name="def_gripper_roll" value="-3.14"/>
 	<xacro:property name="def_gripper_pitch" value="0.0"/>
 	<xacro:property name="def_gripper_yaw" value="0.0"/>
